File: R-CoreLink.kicad_pcb (KiCad board)
At the start: 4 copper layers, 110 x 80 mm, 186 parts, among them IC1 APS6408L-3OC-BA, IC2 AL8866QFN-7, IC5 MCP6n16-100E_MF, IC6 MCP6n16-100E_MF, IC7 MCP6n16-100E_MF, IC8 MCP6n16-100E_MF, J1 541044031, J10 TBC05-03-1-G-G, J11 TBC05-02-1-G-G, J12 TBC05-02-1-G-G, J13 530470410, J14 1734839-6, J19 TBC05-02-1-G-G, J2 RJHSE5384H1, J20 TBC05-02-1-G-G, J21 TBC05-02-1-G-G, J22 TBC05-02-1-G-G, J3 TBC05-03-1-G-G, J4 10155435-00011LF, J5 TBC05-03-1-G-G, J6 TBC05-03-1-G-G, J7 TBC05-03-1-G-G, J8 TBC05-03-1-G-G, J9 TBC05-03-1-G-G, Q1 DMG7430LFG, Q2 IRLML2060, U1 STM32H5E5ZJT6, U11 TCAN3413DRBR, U2 LAN8742A, U3 USBLC6-4SC6, U4 TCPP01-M12, U5 ECMF2-40A100N6, U6 TPS62177DQC, U8 SN65HVD75DRBR, Y1 XC32M4-24.000-F12NJDTL, Y2 LFXTAL009678

Commit message: test
Parts:
- added C56: 100n, Capacitor_SMD:C_0402_1005Metric, F.Cu at (118.5, 50.8)
- added R2: 0, Resistor_SMD:R_0402_1005Metric, F.Cu at (118.5, 48.8)
- added U10: TMUX1108PW, Package_SO:TSSOP-16_4.4x5mm_P0.65mm, F.Cu at (112.7, 57.7)
- added U7: TMUX1108PW, Package_SO:TSSOP-16_4.4x5mm_P0.65mm, F.Cu at (112.7, 51.1)
- moved U3 0.81 mm to (144.7, 84.8)
Routing:
- net +3.3V: track 71.6 -> 70.0 mm
- net /MCU/SRAM_IO5: track 5.58 -> 7.01 mm
